File: KiCad/nano-server/output_2.kicad_sch (KiCad schematic)
At the start: 18 parts, among them J12 OUT_2, J6 SELECT_OUT_2, K10 TIANBO-HJR-4102-L, K3 TIANBO-HJR-4102-L, K4 TIANBO-HJR-4102-L, K5 TIANBO-HJR-4102-L, K6 TIANBO-HJR-4102-L, K7 TIANBO-HJR-4102-L, K8 TIANBO-HJR-4102-L, K9 TIANBO-HJR-4102-L, U10 SN74LVC2G14DBV, U11 SN74LVC2G14DBV, U12 SN74LVC2G14DBV, U13 SN74LVC2G14DBV, U14 ULN2803A, U9 PCF8574T

Commit message: fix schematic and gerbers
Other:
- title: (none) -> Outputs 2
Changed lines of the file:
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@@
 	(generator_version "10.0")
 	(paper "A4")
+	(title_block
+		(title "Outputs 2")
+		(date "2026-08-18")
+	)
 	(text "Near each IC"
 		(exclude_from_sim no)
