File: KiCad/nano-server/outputs.kicad_sch (KiCad schematic)
At the start: 18 parts, among them J11 SELECT_OUT_1, J7 OUT_1, K18 TIANBO-HJR-4102-L, K19 TIANBO-HJR-4102-L, K2 TIANBO-HJR-4102-L, K20 TIANBO-HJR-4102-L, K21 TIANBO-HJR-4102-L, K22 TIANBO-HJR-4102-L, K23 TIANBO-HJR-4102-L, K24 TIANBO-HJR-4102-L, U2 PCF8574T, U3 SN74LVC2G14DBV, U4 SN74LVC2G14DBV, U5 SN74LVC2G14DBV, U6 SN74LVC2G14DBV, U7 ULN2803A

Commit message: fix schematic and gerbers
Other:
- title: (none) -> Outputs 1
Changed lines of the file:
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@@
 	(generator_version "10.0")
 	(paper "A4")
+	(title_block
+		(title "Outputs 1")
+		(date "2026-08-18")
+	)
 	(text "Near each IC"
 		(exclude_from_sim no)
