File: KiCad/nano-server/nano-server.kicad_sch (KiCad schematic)
At the start: 47 parts, among them J1 12-14V, J10 24-27V, J13 MountHole, J14 MountHole, J15 MountHole, J16 MountHole, J17 I2C, J18 CW, J19 UART0, J2 Left_Side, J20 UART1, J3 Right_Side, J4 USB_A, J5 PTT_OUT, K1 TIANBO-HJR-4102-L, Q1 BC817, U1 K7805-500R3, U15 LTV-817S

Commit message: fix schematic and gerbers
Parts:
- added C15, C16, C17, C33: 100n, Capacitor_SMD:C_1206_3216Metric, symbol Device:C
- added U16: MAX232, Package_SO:SOIC-16_3.9x9.9mm_P1.27mm, symbol Interface_UART:MAX232
- J20: value UART1 -> RS232
Connections:
- net +5V: now also C17.2, U16.16 (VCC)
- net GND: now also C33.2, U16.15 (GND)
- net UART1_RX: now also U16.12 (R1OUT); no longer J20.2 (Pin_2)
- net UART1_TX: now also U16.11 (T1IN); no longer J20.3 (Pin_3)
- new net: C16.1, U16.4 (C2+)
- new net: C16.2, U16.5 (C2-)
- new net: C17.1, U16.2 (VS+)
- new net: C15.1, U16.1 (C1+)
- new net: C15.2, U16.3 (C1-)
- new net: C33.1, U16.6 (VS-)
- new net RXD: J20.2 (Pin_2), U16.13 (R1IN)
- new net TXD: J20.3 (Pin_3), U16.14 (T1OUT)
- no-connect marks 19 -> 23
Other:
- title: (none) -> Nano Server for remote operation

Commit message: fix some pcb issues
Parts:
- C4: footprint Capacitor_SMD:C_1206_3216Metric -> Capacitor_SMD:C_1206_3216Metric_Pad1.33x1.80mm_HandSolder
- C9: value 22u -> 10u; footprint Capacitor_SMD:C_1206_3216Metric -> Capacitor_SMD:C_1206_3216Metric_Pad1.33x1.80mm_HandSolder
- D25: footprint Diode_SMD:D_1206_3216Metric -> LED_SMD:LED_1206_3216Metric
- R1, R2, R3, R32, R4: footprint Capacitor_SMD:C_1206_3216Metric -> Resistor_SMD:R_1206_3216Metric
Changed lines of the file:
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@@
 			)
 		)
-		(property "Footprint" "Capacitor_SMD:C_1206_3216Metric"
+		(property "Footprint" "Resistor_SMD:R_1206_3216Metric"
 			(at 83.058 166.37 90)
 			(hide yes)
@@
 			)
 		)
-		(property "Value" "22u"
+		(property "Value" "10u"
 			(at 170.18 31.496 0)
 			(show_name no)
@@
 			)
 		)
-		(property "Footprint" "Capacitor_SMD:C_1206_3216Metric"
+		(property "Footprint" "Capacitor_SMD:C_1206_3216Metric_Pad1.33x1.80mm_HandSolder"
 			(at 169.8752 39.37 0)
 			(hide yes)
@@
 			)
 		)
-		(property "Footprint" "Capacitor_SMD:C_1206_3216Metric"
+		(property "Footprint" "Resistor_SMD:R_1206_3216Metric"
 			(at 127.508 166.37 90)
 			(hide yes)
@@
 			)
 		)
-		(property "Footprint" "Capacitor_SMD:C_1206_3216Metric"
+		(property "Footprint" "Resistor_SMD:R_1206_3216Metric"
 			(at 193.548 97.79 90)
 			(hide yes)
@@
 			)
 		)
-		(property "Footprint" "Capacitor_SMD:C_1206_3216Metric"
+		(property "Footprint" "Capacitor_SMD:C_1206_3216Metric_Pad1.33x1.80mm_HandSolder"
 			(at 116.5352 38.1 0)
 			(hide yes)
@@
 			)
 		)
-		(property "Footprint" "Diode_SMD:D_1206_3216Metric"
+		(property "Footprint" "LED_SMD:LED_1206_3216Metric"
 			(at 125.73 175.26 0)
 			(hide yes)
@@
 			)
 		)
-		(property "Footprint" "Capacitor_SMD:C_1206_3216Metric"
+		(property "Footprint" "Resistor_SMD:R_1206_3216Metric"
 			(at 86.36 163.068 90)
 			(hide yes)
@@
 			)
 		)
-		(property "Footprint" "Capacitor_SMD:C_1206_3216Metric"
+		(property "Footprint" "Resistor_SMD:R_1206_3216Metric"
 			(at 199.898 97.79 90)
 			(hide yes)
