File: KiCad/nano-server/usb_audio.kicad_sch (KiCad schematic)
At the start: 29 parts, among them J8 TO_TRX, J9 FROM_TRX, T1 600:600, T2 600:600, U8 CM108B, Y1 12MHz

Commit message: fix schematic and gerbers
Parts:
- R12, R13: value 470 -> 10
Other:
- title: (none) -> USB Audio
Changed lines of the file:
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@@
 	(generator_version "10.0")
 	(paper "A4")
+	(title_block
+		(title "USB Audio")
+		(date "2026-08-18")
+	)
 	(text "USB Audio"
 		(exclude_from_sim no)
@@
 			)
 		)
-		(property "Value" "470"
+		(property "Value" "10"
 			(at 153.67 82.55 90)
 			(show_name no)
@@
 			)
 		)
-		(property "Value" "470"
+		(property "Value" "10"
 			(at 153.67 87.63 90)
 			(show_name no)

Commit message: fix some pcb issues
Parts:
- C22, C23: footprint Capacitor_SMD:C_1206_3216Metric_Pad1.33x1.80mm_HandSolder -> Capacitor_SMD:C_1206_3216Metric
Changed lines of the file:
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@@
 			)
 		)
-		(property "Footprint" "Capacitor_SMD:C_1206_3216Metric_Pad1.33x1.80mm_HandSolder"
+		(property "Footprint" "Capacitor_SMD:C_1206_3216Metric"
 			(at 135.89 51.1048 0)
 			(hide yes)
@@
 			)
 		)
-		(property "Footprint" "Capacitor_SMD:C_1206_3216Metric_Pad1.33x1.80mm_HandSolder"
+		(property "Footprint" "Capacitor_SMD:C_1206_3216Metric"
 			(at 135.89 58.7248 0)
 			(hide yes)
