File: KiCad/nano-server/nano-server.kicad_pcb (KiCad board)
At the start: 2 copper layers, 144.1 x 108.1 mm, 112 parts, among them J1 12-14V, J10 24-27V, J11 SELECT_OUT_1, J12 OUT_2, J13 MountHole, J14 MountHole, J15 MountHole, J16 MountHole, J17 I2C, J18 CW, J19 UART0, J2 Left_Side, J20 UART1, J3 Right_Side, J4 USB_A, J5 PTT_OUT, J6 SELECT_OUT_2, J7 OUT_1, J8 TO_TRX, J9 FROM_TRX, K1 TIANBO-HJR-4102-L, K10 TIANBO-HJR-4102-L, K18 TIANBO-HJR-4102-L, K19 TIANBO-HJR-4102-L, K2 TIANBO-HJR-4102-L, K20 TIANBO-HJR-4102-L, K21 TIANBO-HJR-4102-L, K22 TIANBO-HJR-4102-L, K23 TIANBO-HJR-4102-L, K24 TIANBO-HJR-4102-L, K3 TIANBO-HJR-4102-L, K4 TIANBO-HJR-4102-L, K5 TIANBO-HJR-4102-L, K6 TIANBO-HJR-4102-L, K7 TIANBO-HJR-4102-L, K8 TIANBO-HJR-4102-L, K9 TIANBO-HJR-4102-L, Q1 BC817, T1 600:600, T2 600:600, U1 K7805-500R3, U10 SN74LVC2G14DBV, U11 SN74LVC2G14DBV, U12 SN74LVC2G14DBV, U13 SN74LVC2G14DBV, U14 ULN2803A, U15 LTV-817S, U2 PCF8574T, U3 SN74LVC2G14DBV, U4 SN74LVC2G14DBV, U5 SN74LVC2G14DBV, U6 SN74LVC2G14DBV, U7 ULN2803A, U8 CM108B, U9 PCF8574T, Y1 12MHz

Commit message: fix schematic and gerbers
Parts:
- added C15: 100n, Capacitor_SMD:C_1206_3216Metric, F.Cu at (78.8, 117.9)
- added C16: 100n, Capacitor_SMD:C_1206_3216Metric, F.Cu at (78.8, 122.9)
- added C17: 100n, Capacitor_SMD:C_1206_3216Metric, F.Cu at (84.5, 117.2)
- added C33: 100n, Capacitor_SMD:C_1206_3216Metric, F.Cu at (78.8, 128.0)
- added U16: MAX232, Package_SO:SOIC-16_3.9x9.9mm_P1.27mm, F.Cu at (84.4, 124.5)
- J20: value UART1 -> RS232
- R12, R13: value 470 -> 10
Connections:
- J20 pad 2: UART1_RX -> RXD
- J20 pad 3: UART1_TX -> TXD
Routing:
- net TXD: track 0.00 -> 28.2 mm, vias 0 -> 1
- net GND: track 713.1 -> 740.3 mm, vias 34 -> 35
- net RXD: track 0.00 -> 24.9 mm, vias 0 -> 1
- net UART1_TX: track 111.7 -> 93.5 mm, vias 3 -> 4
- net UART1_RX: track 110.7 -> 92.7 mm, vias 3 -> 4
- net Net-(U16-VS+): track 0.00 -> 5.90 mm
- net Net-(U16-C1-): track 0.00 -> 5.43 mm
- net PC1: track 116.3 -> 121.3 mm
- net Net-(U16-C1+): track 0.00 -> 4.96 mm
- net Net-(U16-C2+): track 0.00 -> 4.18 mm
- net Net-(U16-C2-): track 0.00 -> 3.49 mm
- net +5V: track 349.2 -> 352.5 mm
- net Net-(U16-VS-): track 0.00 -> 3.18 mm
- net PC2: track 112.0 -> 115.0 mm
- net Net-(T2-SA): track 25.9 -> 26.7 mm
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Other:
- board text added: "RS232"
- board text removed: "UART1"

Commit message: fix some pcb issues
Parts:
- C22, C23: footprint Capacitor_SMD:C_1206_3216Metric_Pad1.33x1.80mm_HandSolder -> Capacitor_SMD:C_1206_3216Metric
- C4: footprint Capacitor_SMD:C_1206_3216Metric -> Capacitor_SMD:C_1206_3216Metric_Pad1.33x1.80mm_HandSolder
- C9: value 22u -> 10u; footprint Capacitor_SMD:C_1206_3216Metric -> Capacitor_SMD:C_1206_3216Metric_Pad1.33x1.80mm_HandSolder
- D25: footprint Diode_SMD:D_1206_3216Metric -> LED_SMD:LED_1206_3216Metric
- R1, R2, R3, R32, R4: footprint Capacitor_SMD:C_1206_3216Metric -> Resistor_SMD:R_1206_3216Metric

Commit message: fix an issue on the board
Routing:
- net +5V: track 352.5 -> 353.9 mm, vias 8 -> 9
Changed lines of the file:
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@@
+	)
+	(segment
+		(start 85.95 117.2)
+		(end 85.89 117.2)
+		(width 0.3)
+		(layer "F.Cu")
+		(net "+5V")
 	)
 	(segment
@@
 		(start 69.4575 93.535)
 		(end 66.7075 93.535)
+		(width 0.3)
+		(layer "F.Cu")
+		(net "+5V")
+	)
+	(segment
+		(start 85.89 117.2)
+		(end 84.89 116.2)
 		(width 0.3)
 		(layer "F.Cu")
@@
 		(net "+5V")
 	)
+	(via
+		(at 84.89 116.2)
+		(size 0.6)
+		(drill 0.3)
+		(layers "F.Cu" "B.Cu")
+		(net "+5V")
+	)
